File: Motor_Controller_Interface/Motor_Controller_Interface_v1_final/Motor_Controller_Interface_v1.kicad_sch (KiCad schematic)
At the start: 13 parts, among them J1 NAV_BOARD_INPUT, J2 RMotor, J3 LMotor, J4 5V POWER, Q1 2N3904, Q2 2N3904, U1 74HCT125

Commit message: finalized resistor values, mounting holes added
Parts:
- R2, R4: value rPull -> 1kΩ
Changed lines of the file:
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@@
 			)
 		)
-		(property "Value" "rPull"
+		(property "Value" "1kΩ"
 			(at 99.06 52.0699 0)
 			(effects
@@
 			)
 		)
-		(property "Value" "rPull"
+		(property "Value" "1kΩ"
 			(at 97.79 81.2799 0)
 			(effects
