File: Motor_Controller_Interface/Motor_Controller_Interface_v1.kicad_pcb (KiCad board)
At the start: 2 copper layers, 67.5 x 45.5 mm, 16 parts, among them J1 NAV_BOARD_INPUT, J2 RMotor, J3 LMotor, J4 5V POWER, Q1 2N3904, Q2 2N3904, U1 74HCT125

Commit message: MCI v1 ordered aug24/2026. JLCPCB approved GBR files
Parts:
- removed the REF** at (188.2, 124.2)
- removed the REF** at (141.0, 118.8)
- removed the REF** at (189.2, 102.0)
- added REF**: MountingHole_2.7mm_M2.5, MountingHole:MountingHole_2.7mm_M2.5, F.Cu at (192.0, 88.0)
- added REF**: MountingHole_2.7mm_M2.5, MountingHole:MountingHole_2.7mm_M2.5, F.Cu at (130.5, 88.0)
- added REF**: MountingHole_2.7mm_M2.5, MountingHole:MountingHole_2.7mm_M2.5, F.Cu at (130.5, 127.6)
- added REF**: MountingHole_2.7mm_M2.5, MountingHole:MountingHole_2.7mm_M2.5, F.Cu at (192.0, 127.5)
- moved J3 6.50 mm to (133.3, 115.0)
- moved J2 6.00 mm to (133.0, 101.0)
- moved J1 5.89 mm to (181.6, 90.4)
- moved C2 3.25 mm to (174.0, 121.2)
- moved J4 3.25 mm to (164.2, 121.2)
Routing:
- net /L_DIR_OUT: track 60.2 -> 52.6 mm
- net /R_DIR: track 43.1 -> 36.4 mm
- net /R_SPEED: track 59.0 -> 52.8 mm
- net /L_DIR: track 52.9 -> 47.0 mm
- net /L_SPEED: track 72.5 -> 66.8 mm
- net /R_SPEED_OUT: track 46.5 -> 41.9 mm
- net +5V: track 109.3 -> 106.1 mm
- net /R_DIR_OUT: track 28.2 -> 30.7 mm
- net /L_SPEED_OUT: track 38.5 -> 36.2 mm
